File: Schématique Harpe/Schématique Harpe.kicad_sch (KiCad schematic)
At the start: 34 parts, among them IC1 VL53L8CXV9GC_1, J1 USB_C_Receptacle_USB2.0_16P, U1 STM32G431KBTx, U2 PAM8403DR, U3 USBLC6-2SC6, U4 TXS0102DCT

Commit message: Add files via upload
Parts:
- removed U4: TXS0102DCT, Package_SO:SSOP-8_2.95x2.8mm_P0.65mm, symbol Logic_LevelTranslator:TXS0102DCT
- added C14: 1uF, symbol Device:C_Small
- added D1, D2: LED, symbol Device:LED
- added R12: R, symbol Device:R
- added U4: AP2112K-1.8, Package_TO_SOT_SMD:SOT-23-5, symbol Regulator_Linear:AP2112K-1.8
- C6: value 0.47uF -> 1uF
- IC1: footprint VL53L8CXV9GC1 -> composant:VL53L8CXV9GC1
- PS1: footprint BU33SD5WG-TR:SOT95P280X125-5N -> composant:BU33SD5WG-TR
- R3: value Ri -> R
- R4: value Ri -> 18k
Connections:
- net INR is gone; now on net GND: C6.1
- net +3.3V: now also C6.2, U4.1 (VIN); no longer U1.15 (VDDA)
- net GND: now also U1.14 (VSSA), U1.16 (VSS), U1.32 (VSS), C14.1, U4.2 (GND)
- net INL: now also U1.9 (PA4)
- net IOVDD: now also C14.2, U4.5 (VOUT)
- net MUTE: now also U1.11 (PA6)
- net NCS: now also U1.8 (PA3)
- net SHDN: now also U1.10 (PA5)
- net STBY: now also U1.12 (PA7)
- net at U2.10 (INR): no longer R3.1
- net at R3.2: no longer C6.2
- new net: D2.2 (A), R3.1
- new net: D1.2 (A), R12.2
- new net +3.3VA: U1.15 (VDDA)
- no-connect marks 6 -> 21
Other:
- note added: "Adaptateur de niveaux"
- note added: "Connecteur et autres"
- moved on the sheet: R11

Commit message: Add files via upload
Parts:
- added U5: ACPL-M61L-000E, ACPL-M61L-000E:ACPL-M61L-000E, symbol ACPL-M61L-000E:ACPL-M61L-000E
Connections:
- net +3.3VA is gone; now on net IOVDD: U1.15 (VDDA)
- net +3.3V: no longer U1.1 (VDD), U1.17 (VDD)
- net IOVDD: now also U1.1 (VDD), U1.17 (VDD)
Other:
- note added: "midi"
- note removed: "Adaptateur de niveaux"
